Commit message: 清理 TurtleBot3 的 Gazebo 参数并修正网格模型路径
- 删除 TurtleBot3 差速驱动 Gazebo 插件中不受支持的 odometry_source 配置
- 将 TurtleBot3 的网格模型引用从 package://sim_env/... 改为 file:///...，避免生成机器人时依赖扩大的 GAZEBO_MODEL_PATH
- 统一 burger、waffle 和 waffle_pi 三种机器人在 ROS 2 + Gazebo Classic 下的描述写法

File: sim_env/urdf/turtlebot3_burger/turtlebot3_burger.gazebo.xacro (robot description, xacro)
@@ -60,5 +60,4 @@
       <odometry_frame>odom</odometry_frame>
       <robot_base_frame>base_footprint</robot_base_frame>
-      <odometry_source>world</odometry_source>
       <publish_odom>true</publish_odom>
       <publish_odom_tf>true</publish_odom_tf>

File: sim_env/urdf/turtlebot3_burger/turtlebot3_burger.urdf.xacro (robot description, xacro)
@@ -11,5 +11,5 @@
       <origin xyz="-0.032 0 0.0" rpy="0 0 0" />
       <geometry>
-        <mesh filename="package://sim_env/meshes/turtlebot3/bases/burger_base.stl" scale="0.001 0.001 0.001" />
+        <mesh filename="file://$(find sim_env)/meshes/turtlebot3/bases/burger_base.stl" scale="0.001 0.001 0.001" />
       </geometry>
       <material name="light_black" />
@@ -39,5 +39,5 @@
       <origin xyz="0 0 0" rpy="1.57 0 0" />
       <geometry>
-        <mesh filename="package://sim_env/meshes/turtlebot3/wheels/left_tire.stl" scale="0.001 0.001 0.001" />
+        <mesh filename="file://$(find sim_env)/meshes/turtlebot3/wheels/left_tire.stl" scale="0.001 0.001 0.001" />
       </geometry>
       <material name="dark" />
@@ -67,5 +67,5 @@
       <origin xyz="0 0 0" rpy="1.57 0 0" />
       <geometry>
-        <mesh filename="package://sim_env/meshes/turtlebot3/wheels/right_tire.stl" scale="0.001 0.001 0.001" />
+        <mesh filename="file://$(find sim_env)/meshes/turtlebot3/wheels/right_tire.stl" scale="0.001 0.001 0.001" />
       </geometry>
       <material name="dark" />
@@ -120,5 +120,5 @@
       <origin xyz="0 0 0.0" rpy="0 0 0" />
       <geometry>
-        <mesh filename="package://sim_env/meshes/turtlebot3/sensors/lds.stl" scale="0.001 0.001 0.001" />
+        <mesh filename="file://$(find sim_env)/meshes/turtlebot3/sensors/lds.stl" scale="0.001 0.001 0.001" />
       </geometry>
       <material name="dark" />

File: sim_env/urdf/turtlebot3_waffle/turtlebot3_waffle.gazebo.xacro (robot description, xacro)
@@ -129,5 +129,4 @@
       <odometry_frame>odom</odometry_frame>
       <robot_base_frame>base_footprint</robot_base_frame>
-      <odometry_source>world</odometry_source>
       <publish_odom>true</publish_odom>
       <publish_odom_tf>true</publish_odom_tf>

File: sim_env/urdf/turtlebot3_waffle/turtlebot3_waffle.urdf.xacro (robot description, xacro)
@@ -15,5 +15,5 @@
       <origin xyz="-0.064 0 0.0" rpy="0 0 0" />
       <geometry>
-        <mesh filename="package://sim_env/meshes/turtlebot3/bases/waffle_base.stl" scale="0.001 0.001 0.001" />
+        <mesh filename="file://$(find sim_env)/meshes/turtlebot3/bases/waffle_base.stl" scale="0.001 0.001 0.001" />
       </geometry>
       <material name="light_black" />
@@ -43,5 +43,5 @@
       <origin xyz="0 0 0" rpy="1.57 0 0" />
       <geometry>
-        <mesh filename="package://sim_env/meshes/turtlebot3/wheels/left_tire.stl" scale="0.001 0.001 0.001" />
+        <mesh filename="file://$(find sim_env)/meshes/turtlebot3/wheels/left_tire.stl" scale="0.001 0.001 0.001" />
       </geometry>
       <material name="dark" />
@@ -71,5 +71,5 @@
       <origin xyz="0 0 0" rpy="1.57 0 0" />
       <geometry>
-        <mesh filename="package://sim_env/meshes/turtlebot3/wheels/right_tire.stl" scale="0.001 0.001 0.001" />
+        <mesh filename="file://$(find sim_env)/meshes/turtlebot3/wheels/right_tire.stl" scale="0.001 0.001 0.001" />
       </geometry>
       <material name="dark" />
@@ -144,5 +144,5 @@
       <origin xyz="0 0 0" rpy="0 0 0" />
       <geometry>
-        <mesh filename="package://sim_env/meshes/turtlebot3/sensors/lds.stl" scale="0.001 0.001 0.001" />
+        <mesh filename="file://$(find sim_env)/meshes/turtlebot3/sensors/lds.stl" scale="0.001 0.001 0.001" />
       </geometry>
       <material name="dark" />
@@ -171,5 +171,5 @@
       <origin xyz="0 0 0" rpy="1.57 0 1.57" />
       <geometry>
-        <mesh filename="package://sim_env/meshes/turtlebot3/sensors/r200.dae" />
+        <mesh filename="file://$(find sim_env)/meshes/turtlebot3/sensors/r200.dae" />
       </geometry>
     </visual>

File: sim_env/urdf/turtlebot3_waffle_pi/turtlebot3_waffle_pi.gazebo.xacro (robot description, xacro)
@@ -70,5 +70,4 @@
       <odometry_frame>odom</odometry_frame>
       <robot_base_frame>base_footprint</robot_base_frame>
-      <odometry_source>world</odometry_source>
       <publish_odom>true</publish_odom>
       <publish_odom_tf>true</publish_odom_tf>

File: sim_env/urdf/turtlebot3_waffle_pi/turtlebot3_waffle_pi.urdf.xacro (robot description, xacro)
@@ -11,5 +11,5 @@
       <origin xyz="-0.064 0 0.0" rpy="0 0 0" />
       <geometry>
-        <mesh filename="package://sim_env/meshes/turtlebot3/bases/waffle_pi_base.stl" scale="0.001 0.001 0.001" />
+        <mesh filename="file://$(find sim_env)/meshes/turtlebot3/bases/waffle_pi_base.stl" scale="0.001 0.001 0.001" />
       </geometry>
       <material name="light_black" />
@@ -39,5 +39,5 @@
       <origin xyz="0 0 0" rpy="1.57 0 0" />
       <geometry>
-        <mesh filename="package://sim_env/meshes/turtlebot3/wheels/left_tire.stl" scale="0.001 0.001 0.001" />
+        <mesh filename="file://$(find sim_env)/meshes/turtlebot3/wheels/left_tire.stl" scale="0.001 0.001 0.001" />
       </geometry>
       <material name="dark" />
@@ -67,5 +67,5 @@
       <origin xyz="0 0 0" rpy="1.57 0 0" />
       <geometry>
-        <mesh filename="package://sim_env/meshes/turtlebot3/wheels/right_tire.stl" scale="0.001 0.001 0.001" />
+        <mesh filename="file://$(find sim_env)/meshes/turtlebot3/wheels/right_tire.stl" scale="0.001 0.001 0.001" />
       </geometry>
       <material name="dark" />
@@ -140,5 +140,5 @@
       <origin xyz="0 0 0.0" rpy="0 0 0" />
       <geometry>
-        <mesh filename="package://sim_env/meshes/turtlebot3/sensors/lds.stl" scale="0.001 0.001 0.001" />
+        <mesh filename="file://$(find sim_env)/meshes/turtlebot3/sensors/lds.stl" scale="0.001 0.001 0.001" />
       </geometry>
       <material name="dark" />
